File: T03_Eagle_Files/T03_MotionControledLamp.brd (EAGLE design)
At the start: 17.8 x 30.5 mm, 32 parts, among them SW1 RESET, U1 ATMEGA328P-MU, U2 V_REG_LD1085D2, U4 TPS61161ADRVT, X2 16MHz

Commit message: Implementing Feedback
Parts:
- removed R2: 10K, Smartprj:R0603-ROUND
- removed U$11: DISCLAIMER, Smartprj:DISCLAIMER
- removed U2: V_REG_LD1085D2, SparkFun-PowerIC:D2PACK/A
- added IC1: L7805, v-reg:78XXL
- added JP2: BAT_POS_VOLT, adafruit:1X01
- added JP3: BAT_GND, adafruit:1X01
- added R3: 10k, rcl:M1206
- C5: value 100uF -> 10uF
- C6: value 0.1uF -> 1uF
- C9: value 0.1uF -> 220nF
- D1: value 3.3V -> 0.2V
- L1: value (none) -> 22uH
- R1: value (none) -> 10
Connections:
- net IO10 renamed PWM_LEDS
- net IO11 renamed MOSI
- net IO12 renamed MISO
- removed net ADC0: U1.23
- removed net ADC1: U1.24
- removed net ADC2: U1.25
- removed net ADC3: U1.26
- removed net ADC4: U1.27
- removed net ADC5: U1.28
- removed net ADC6: U1.19
- removed net ADC7: U1.22
- removed net IO2: U1.32
- removed net IO3: U1.1
- removed net IO4: U1.2
- removed net IO5: U1.9
- removed net IO6: U1.10
- removed net IO7: U1.11
- removed net IO8: U1.12
- removed net IO9: U1.13
- removed net N$5: U1.17
- removed net VCC: PWR_SWTCH.P
- new net +V_BAT: JP2.1, PWR_SWTCH.P
- new net N$11: LED5.C, LED5.C@1, LED5.C@2, LED5.C@3, LED5.C@4, LED5.C@5, LED8.A
- new net N$12: LED3.A, LED6.C, LED6.C@1, LED6.C@2, LED6.C@3, LED6.C@4, LED6.C@5
- new net N$15: LED4.C, LED4.C@1, LED4.C@2, LED4.C@3, LED4.C@4, LED4.C@5, LED7.A
- new net NC: U1.1, U1.10, U1.11, U1.12, U1.13, U1.19, U1.2, U1.22, U1.23, U1.24, U1.25, U1.26, U1.27, U1.28, U1.32, U1.9
- net +5V: now also IC1.OUT, R3.2; no longer R2.2, U2.2, U2.TAB
- net GND: now also IC1.GND, JP1.4, JP3.1; no longer U2.1
- net N$14: no longer LED5.C, LED5.C@1, LED5.C@2, LED5.C@3, LED5.C@4, LED5.C@5
- net N$4: now also IC1.IN; no longer U2.3
- net N$9: now also LED6.A; no longer LED3.A, LED4.C, LED4.C@1, LED4.C@2, LED4.C@3, LED4.C@4, LED4.C@5
- net RST: now also JP1.7, R3.1, U1.17; no longer R2.1
Routing:
- net NC: track 0.00 -> 140.3 mm, vias 0 -> 4
- net ADC5: track 18.5 -> 0.00 mm, vias 1 -> 0
- net ADC4: track 17.7 -> 0.00 mm, vias 1 -> 0
- net IO9: track 13.9 -> 0.00 mm
- net IO8: track 11.9 -> 0.00 mm
- net ADC7: track 11.4 -> 0.00 mm, vias 1 -> 0
- net ADC6: track 9.72 -> 0.00 mm, vias 1 -> 0
- net IO7: track 9.27 -> 0.00 mm
- net ADC3: track 7.27 -> 0.00 mm
- net IO2: track 6.45 -> 0.00 mm
- net ADC0: track 6.01 -> 0.00 mm
- net IO6: track 5.96 -> 0.00 mm
- net IO5: track 5.59 -> 0.00 mm
- net ADC2: track 4.75 -> 0.00 mm
- net IO3: track 4.55 -> 0.00 mm
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